Commit message: Update wx250s.urdf.xacro

File: interbotix_ros_xsarms/interbotix_xsarm_descriptions/urdf/wx250s.urdf.xacro (robot description, xacro)
@@ -17,4 +17,13 @@
     <texture filename="package://interbotix_xsarm_descriptions/meshes/interbotix_black.png"/>
   </material>
+  <material name="dark_blue">
+    <color rgba="0.2 0.3 0.36 1"/>
+  </material>
+  <material name="blue">
+    <color rgba="0.11 0.36 0.53 1"/>
+  </material>
+  <material name="green">
+    <color rgba="0.33 0.67 0.47 1"/>
+  </material>
   <xacro:if value="$(arg use_world_frame)">
     <link name="world"/>
@@ -30,5 +39,5 @@
         <mesh filename="package://interbotix_xsarm_descriptions/meshes/wx250s_meshes/wx250s_1_base.stl" scale="0.001 0.001 0.001"/>
       </geometry>
-      <material name="interbotix_black"/>
+      <material name="dark_blue"/>
     </visual>
     <collision>
@@ -67,5 +76,5 @@
         <mesh filename="package://interbotix_xsarm_descriptions/meshes/wx250s_meshes/wx250s_2_shoulder.stl" scale="0.001 0.001 0.001"/>
       </geometry>
-      <material name="interbotix_black"/>
+      <material name="green"/>
     </visual>
     <collision>
@@ -104,5 +113,5 @@
         <mesh filename="package://interbotix_xsarm_descriptions/meshes/wx250s_meshes/wx250s_3_upper_arm.stl" scale="0.001 0.001 0.001"/>
       </geometry>
-      <material name="interbotix_black"/>
+      <material name="dark_blue"/>
     </visual>
     <collision>
@@ -141,5 +150,5 @@
         <mesh filename="package://interbotix_xsarm_descriptions/meshes/wx250s_meshes/wx250s_4_upper_forearm.stl" scale="0.001 0.001 0.001"/>
       </geometry>
-      <material name="interbotix_black"/>
+      <material name="green"/>
     </visual>
     <collision>
@@ -178,5 +187,5 @@
         <mesh filename="package://interbotix_xsarm_descriptions/meshes/wx250s_meshes/wx250s_5_lower_forearm.stl" scale="0.001 0.001 0.001"/>
       </geometry>
-      <material name="interbotix_black"/>
+      <material name="dark_blue"/>
     </visual>
     <collision>
@@ -215,5 +224,5 @@
         <mesh filename="package://interbotix_xsarm_descriptions/meshes/wx250s_meshes/wx250s_6_wrist.stl" scale="0.001 0.001 0.001"/>
       </geometry>
-      <material name="interbotix_black"/>
+      <material name="green"/>
     </visual>
     <collision>
@@ -252,5 +261,5 @@
         <mesh filename="package://interbotix_xsarm_descriptions/meshes/wx250s_meshes/wx250s_7_gripper.stl" scale="0.001 0.001 0.001"/>
       </geometry>
-      <material name="interbotix_black"/>
+      <material name="dark_blue"/>
     </visual>
     <collision>
@@ -301,5 +310,5 @@
         <mesh filename="package://interbotix_xsarm_descriptions/meshes/wx250s_meshes/wx250s_8_gripper_prop.stl" scale="0.001 0.001 0.001"/>
       </geometry>
-      <material name="interbotix_black"/>
+      <material name="green"/>
     </visual>
     <collision>
@@ -329,5 +338,5 @@
           <mesh filename="package://interbotix_xsarm_descriptions/meshes/wx250s_meshes/wx250s_11_ar_tag.stl" scale="0.001 0.001 0.001"/>
         </geometry>
-        <material name="interbotix_black"/>
+        <material name="dark_blue"/>
       </visual>
       <collision>
@@ -358,5 +367,5 @@
           <mesh filename="package://interbotix_xsarm_descriptions/meshes/wx250s_meshes/wx250s_9_gripper_bar.stl" scale="0.001 0.001 0.001"/>
         </geometry>
-        <material name="interbotix_black"/>
+        <material name="green"/>
       </visual>
       <collision>
@@ -409,5 +418,5 @@
             <mesh filename="package://interbotix_xsarm_descriptions/meshes/wx250s_meshes/wx250s_10_gripper_finger.stl" scale="0.001 0.001 0.001"/>
           </geometry>
-          <material name="interbotix_black"/>
+          <material name="dark_blue"/>
         </visual>
         <collision>
@@ -449,5 +458,5 @@
             <mesh filename="package://interbotix_xsarm_descriptions/meshes/wx250s_meshes/wx250s_10_gripper_finger.stl" scale="0.001 0.001 0.001"/>
           </geometry>
-          <material name="interbotix_black"/>
+          <material name="dark_blue"/>
         </visual>
         <collision>
